Commit message: add function to control dynx joint angle

File: ros/dynamixel_description/urdf/_2XL430.gazebo.xacro (robot description, xacro)
@@ -1,6 +1,17 @@
 <?xml version="1.0"?>
 <!-- あとでdynamixel descriptionを作ってそこにれる -->
-<robot name=" dynamixel-2XL430" xmlns:xacro="http://ros.org/wiki/xacro">\
-	<!--あとでgazebo.xacroに入れる-->
+<robot name="dynamixel-2XL430" xmlns:xacro="http://ros.org/wiki/xacro">\
+	<!-- Transmission macro -->
+	<xacro:macro name="SimpleTransmissionPosition" params="joint motor">
+		<transmission name="tran_${joint}">
+			<type>transmission_interface/SimpleTransmission</type>
+			<joint name="${joint}">
+			<hardwareInterface>hardware_interface/PositionJointInterface</hardwareInterface>
+			</joint>
+			<actuator name="${motor}">
+			<mechanicalReduction>1</mechanicalReduction>
+			</actuator>
+		</transmission>
+	</xacro:macro>
 	<gazebo reference="dynx_2XL430">
 		<mu1>0.1</mu1>
@@ -13,3 +24,17 @@
 		<material>Gazebo/Gray</material>
 	</gazebo>
+	<xacro:SimpleTransmissionPosition motor="dynx_motor1" joint="${parent}_joint" />
+	<xacro:SimpleTransmissionPosition motor="dynx_motor2" joint="${child}_joint" />
+    <!--ros_controlプラグインをロード-->
+    <gazebo>
+      <plugin name="control" filename="libgazebo_ros_control.so">
+		 <!-- <robotNamespace>/dynamixel-2XL430</robotNamespace> -->
+		 <!-- これあるとうまくいかん -->
+		</plugin>
+    </gazebo>
+    <gazebo>
+      <plugin name="joint_state_publisher" filename="libgazebo_ros_joint_state_publisher.so">
+         <jointName>${parent}_joint, ${child}_joint</jointName>
+      </plugin>
+    </gazebo>
 </robot>

File: ros/dynamixel_description/urdf/test_2XL430_servo.urdf.xacro (robot description, xacro)
@@ -22,4 +22,26 @@
 		</visual>
 	</link>
+	<link name="weight">
+		<visual>
+			<origin xyz="0 0 0" rpy="0 0 0"/>
+			<geometry>
+				<box size="0.01 0.01 0.01"/>
+			</geometry>
+			<material name="red"/>
+		</visual>
+		<inertial>
+			<origin xyz="0 0 0" rpy="0 0 0" />
+			<mass value="0.1" />
+			<inertia
+				ixx="0.01" ixy="0.0" ixz="0.0"
+				iyy="0.01" iyz="0.0"
+				izz="0.01" />
+		</inertial>
+	</link>
+	<joint name="fix_wight" type="fixed">
+		<parent link="hone"/>
+		<child link="weight"/>
+		<origin xyz="0 0.05 0" rpy="0 0 0"/>
+	</joint>
 	<gazebo reference="base">
 		<material>Gazebo/Orange</material>

Commit message: update dynamixel 2XL430

File: ros/dynamixel_description/urdf/_2XL430.gazebo.xacro (robot description, xacro)
@@ -7,8 +7,8 @@
 			<type>transmission_interface/SimpleTransmission</type>
 			<joint name="${joint}">
-			<hardwareInterface>hardware_interface/PositionJointInterface</hardwareInterface>
+			    <hardwareInterface>hardware_interface/PositionJointInterface</hardwareInterface>
 			</joint>
 			<actuator name="${motor}">
-			<mechanicalReduction>1</mechanicalReduction>
+			    <mechanicalReduction>1</mechanicalReduction>
 			</actuator>
 		</transmission>
@@ -28,10 +28,4 @@
     <!--ros_controlプラグインをロード-->
     <gazebo>
-      <plugin name="control" filename="libgazebo_ros_control.so">
-		 <!-- <robotNamespace>/dynamixel-2XL430</robotNamespace> -->
-		 <!-- これあるとうまくいかん -->
-		</plugin>
-    </gazebo>
-    <gazebo>
       <plugin name="joint_state_publisher" filename="libgazebo_ros_joint_state_publisher.so">
          <jointName>${parent}_joint, ${child}_joint</jointName>

File: ros/dynamixel_description/urdf/_2XL430.urdf.xacro (robot description, xacro)
@@ -47,5 +47,5 @@
 			<child link="dynx_2XL430"/>
 			<origin xyz="${L_x_yaw} ${L_y_yaw} ${L_z_yaw}" rpy="${pi} 0 0"/>
-			<axis xyz="0 0 1"/>
+			<axis xyz="0 0 -1"/>
 			<dynamics damping="0.1"/>
 			<limit velocity="${no_load_speed}" effort="${stall_torque}" />
@@ -77,5 +77,5 @@
 			<parent link="dynx_2XL430"/>
 			<child link="dynx_2XL430_hone_pitch"/>
-			<origin xyz="${L_x_pitch} ${L_y_pitch} ${L_z_pitch}" rpy="0 ${pi/2} 0"/>
+			<origin xyz="${L_x_pitch} ${L_y_pitch} ${L_z_pitch}" rpy="${0} ${pi/2} ${0}"/>
 			<axis xyz="0 0 1"/>
 			<dynamics damping="0.1"/>

File: ros/dynamixel_description/urdf/test_2XL430_servo.urdf.xacro (robot description, xacro)
@@ -50,3 +50,8 @@
 		<material>Gazebo/Red</material>
 	</gazebo>
+    <!--ros_controlプラグインをロード-->
+    <gazebo>
+        <plugin name="control" filename="libgazebo_ros_control.so">
+        </plugin>
+    </gazebo>
 </robot>
