Commit message: adjust parameters

File: ros/dynamixel_description/urdf/_XM430.urdf.xacro (robot description, xacro)
@@ -11,5 +11,5 @@
         <xacro:include filename="$(find dynamixel_description)/urdf/_XM430.gazebo.xacro"/>
         <!-- STL, daeファイルへの相対パス -->
-		<xacro:property name="path_to_mesh" value="meshes/XM430_idler.stl" />
+		<xacro:property name="path_to_mesh" value="meshes/XM430_W210-R.stl" />
         <!-- 各辺の中点が原点となるように変換 -->
 		<xacro:property name="visual_origin"> <origin xyz="${0} ${L_y_hone} ${0}" rpy="${0} ${0} ${0}" /> </xacro:property>
@@ -21,11 +21,11 @@
 		<xacro:property name="W_y" value="${46.5/1000}" /> <!-- unit [m] --> <!-- converted from [mm] -->
 		<xacro:property name="W_z" value="${34.0/1000}" /> <!-- unit [m] --> <!-- converted from [mm] -->
-		<xacro:property name="no_load_speed" value="${66*(2*pi/60)}" /> <!-- unit [rad/sec] --> <!-- converted from [rev/min] -->
-		<xacro:property name="stall_torque"  value="${8.9}" /> <!-- unit [Nm] -->
-		<xacro:property name="mass"  value="${165/1000}" /> <!-- unit [kg] --> <!-- converted from [g] -->
+		<xacro:property name="no_load_speed" value="${77*(2*pi/60)}" /> <!-- unit [rad/sec] --> <!-- converted from [rev/min] -->
+		<xacro:property name="stall_torque"  value="${3.0}" /> <!-- unit [Nm] -->
+		<xacro:property name="mass"  value="${ 82/1000}" /> <!-- unit [kg] --> <!-- converted from [g] -->
 		<xacro:property name="inertia"> <!-- unit [kg*m^@] --> <!-- converted from [g*mm^2] -->
-			<inertia ixx="${72456.754/1000000000}"  ixy="${-128.62012/1000000000}" ixz="${-174.27089/1000000000}"
-			                                        iyy="${ 38622.228/1000000000}" iyz="${-8272.2282/1000000000}"
-			                                                                       izz="${ 60707.131/1000000000}" />
+			<inertia ixx="${23463.440/1000000000}"  ixy="${-119.06520/1000000000}" ixz="${-64.694734/1000000000}"
+			                                        iyy="${ 12822.944/1000000000}" iyz="${-1799.5812/1000000000}"
+			                                                                       izz="${ 21008.291/1000000000}" />
 		</xacro:property>
 		<joint name="${joint_name}_XM430_base_connector_" type="fixed">
