Commit message: debug the issue of "no show in gazebo"

File: ros/dynamixel_description/urdf/_2XL430.urdf.xacro (robot description, xacro)
@@ -33,6 +33,15 @@
 			</xacro:unless>
 		</joint>
-		<link name="dynx_2XL430_hone_yaw" />
-		<joint name="${parent}_joint" type="fixed">
+		<link name="dynx_2XL430_hone_yaw">
+			<inertial>
+			<origin xyz="0 0 0" rpy="0 0 0" />
+			<mass value="0.00001" />
+			<inertia
+				ixx="0.00001" ixy="0.0" ixz="0.0"
+				iyy="0.00001" iyz="0.0"
+				izz="0.00001" />
+			</inertial>
+		</link>
+		<joint name="${parent}_joint" type="continuous">
 			<parent link="dynx_2XL430_hone_yaw"/>
 			<child link="dynx_2XL430"/>
@@ -65,5 +74,5 @@
 			</collision>
 		</link>
-		<joint name="${child}_joint" type="fixed">
+		<joint name="${child}_joint" type="continuous">
 			<parent link="dynx_2XL430"/>
 			<child link="dynx_2XL430_hone_pitch"/>
@@ -73,5 +82,14 @@
 			<limit velocity="${no_load_speed}" effort="${stall_torque}" />
 		</joint>
-		<link name="dynx_2XL430_hone_pitch" />
+		<link name="dynx_2XL430_hone_pitch">
+			<inertial>
+			<origin xyz="0 0 0" rpy="0 0 0" />
+			<mass value="0.00001" />
+			<inertia
+				ixx="0.00001" ixy="0.0" ixz="0.0"
+				iyy="0.00001" iyz="0.0"
+				izz="0.00001" />
+			</inertial>
+		</link>
 		<joint name="2XL430_pitch_joint_" type="fixed">
 			<parent link="dynx_2XL430_hone_pitch"/>

Commit message: bug fix

File: ros/dynamixel_description/urdf/_2XL430.urdf.xacro (robot description, xacro)
@@ -9,5 +9,5 @@
 		<xacro:property name="L_y_yaw" value="${12/1000}" /> <!-- unit [m] --> <!-- converted from [mm] -->
 		<xacro:property name="L_z_yaw" value="${19/1000}" /> <!-- unit [m] --> <!-- converted from [mm] -->
-		<xacro:property name="L_x_pitch" value="${ L_z_yaw}" /> <!-- unit [m] -->
+		<xacro:property name="L_x_pitch" value="${-L_z_yaw}" /> <!-- unit [m] -->
 		<xacro:property name="L_y_pitch" value="${-L_y_yaw}" /> <!-- unit [m] -->
 		<xacro:property name="L_z_pitch" value="${ L_x_yaw}" /> <!-- unit [m] -->
@@ -46,6 +46,5 @@
 			<parent link="dynx_2XL430_hone_yaw"/>
 			<child link="dynx_2XL430"/>
-			<origin xyz="${L_x_yaw} ${L_y_yaw} ${L_z_yaw}" rpy="${pi} 0 0"/>
-			<axis xyz="0 0 -1"/>
+			<axis xyz="0 0 1"/>
 			<dynamics damping="0.1"/>
 			<limit velocity="${no_load_speed}" effort="${stall_torque}" />
@@ -53,10 +52,10 @@
 		<link name="dynx_2XL430">
 			<inertial>
-				<origin xyz="0 0 0" rpy="0 0 0"/>
+			    <origin xyz="${L_x_yaw} ${L_y_yaw} ${L_z_yaw}" rpy="${pi} 0 0"/>
 				<mass value="${mass}"/>
 				<xacro:insert_block name="inertia"/>
 			</inertial>
 			<visual>
-				<xacro:insert_block name="visual_origin"/>
+                <origin xyz="${L_x_yaw} ${L_y_yaw} ${L_z_yaw}" rpy="${pi} 0 0"/>
 				<geometry>
 					<mesh filename="package://dynamixel_description/${path_to_mesh}" />
@@ -67,5 +66,5 @@
 			</visual>
 			<collision>
-				<origin xyz="0 0 0" rpy="0 0 0"/>
+			    <origin xyz="${L_x_yaw} ${L_y_yaw} ${L_z_yaw}" rpy="${pi} 0 0"/>
 				<geometry>
 					<box size="${W_x} ${W_y} ${W_z}"/>
@@ -77,6 +76,6 @@
 			<parent link="dynx_2XL430"/>
 			<child link="dynx_2XL430_hone_pitch"/>
-			<origin xyz="${L_x_pitch} ${L_y_pitch} ${L_z_pitch}" rpy="${0} ${pi/2} ${0}"/>
-			<axis xyz="0 0 1"/>
+			<origin xyz="${L_x_yaw-L_x_pitch} ${L_y_yaw-L_y_pitch} ${L_z_yaw-L_z_pitch}" rpy="${pi} 0 0"/>
+			<axis xyz="1 0 0"/>
 			<dynamics damping="0.1"/>
 			<limit velocity="${no_load_speed}" effort="${stall_torque}" />
@@ -96,8 +95,8 @@
 			<child link="${child}"/>
 			<xacro:if value="${center_child}">
-				<origin xyz="0 0 ${-L_x_pitch}" rpy="0 0 0"/>
+				<origin xyz="${L_x_pitch} 0 0" rpy="0 ${pi/2} 0"/>
 			</xacro:if>
 			<xacro:unless value="${center_child}">
-				<origin xyz="0 0 0" rpy="0 0 0"/>
+				<origin xyz="0 0 0" rpy="0 ${pi/2} 0"/>
 			</xacro:unless>
 		</joint>

File: ros/dynamixel_description/urdf/test_2XL430_servo.urdf.xacro (robot description, xacro)
@@ -12,5 +12,5 @@
 		</visual>
 	</link>
-	<xacro:servo_2XL430 parent="base" center_parent="false" child="hone" center_child="true" />
+	<xacro:servo_2XL430 parent="base" center_parent="true" child="hone" center_child="true" />
 	<link name="hone">
 		<visual>
