Commit message: update dynamixel XM540

File: ros/dynamixel_description/urdf/_XM540.gazebo.xacro (robot description, xacro)
@@ -1,7 +1,18 @@
 <?xml version="1.0"?>
 <!-- あとでdynamixel descriptionを作ってそこにれる -->
-<robot name=" dynamixel-XM540" xmlns:xacro="http://ros.org/wiki/xacro">\
-	<!--あとでgazebo.xacroに入れる-->
-	<gazebo reference="dynx_XM540">
+<robot name="dynamixel-XM540" xmlns:xacro="http://ros.org/wiki/xacro">\
+	<!-- Transmission macro -->
+	<xacro:macro name="SimpleTransmissionPosition" params="joint motor">
+		<transmission name="tran_${joint}">
+			<type>transmission_interface/SimpleTransmission</type>
+			<joint name="${joint}">
+			<hardwareInterface>hardware_interface/PositionJointInterface</hardwareInterface>
+			</joint>
+			<actuator name="${motor}">
+			<mechanicalReduction>1</mechanicalReduction>
+			</actuator>
+		</transmission>
+	</xacro:macro>
+	<gazebo reference="${joint_name}_dynx_XM540">
 		<mu1>0.1</mu1>
 		<mu2>0.1</mu2>
@@ -13,3 +24,9 @@
 		<material>Gazebo/Gray</material>
 	</gazebo>
+	<xacro:SimpleTransmissionPosition motor="${joint_name}_dynx_motor" joint="${joint_name}_joint" />
+    <gazebo>
+      <plugin name="joint_state_publisher" filename="libgazebo_ros_joint_state_publisher.so">
+        <jointName>${joint_name}_joint</jointName>
+      </plugin>
+    </gazebo>
 </robot>

File: ros/dynamixel_description/urdf/_XM540.urdf.xacro (robot description, xacro)
@@ -2,8 +2,17 @@
 <!-- あとでdynamixel descriptionを作ってそこにれる -->
 <robot name=" dynamixel-XM540" xmlns:xacro="http://ros.org/wiki/xacro">\
-	<xacro:macro name="servo_XM540" params="parent child fixed_plane:=bottom center_child:=false">
-	   <xacro:include filename="$(find dynamixel_description)/urdf/_XM540.gazebo.xacro"/>
+	<xacro:macro name="servo_XM540" params="name:='__defalut__' parent child fixed_plane:=bottom fixed_angle:=0 center_child:=false">
+        <xacro:if value="${name == '__defalut__'}">
+		    <xacro:property name="joint_name" value="${child}" />
+        </xacro:if>
+        <xacro:unless value="${name == '__defalut__'}">
+		    <xacro:property name="joint_name" value="${name}" />
+        </xacro:unless>
+        <xacro:include filename="$(find dynamixel_description)/urdf/_XM540.gazebo.xacro"/>
+        <!-- STL, daeファイルへの相対パス -->
 		<xacro:property name="path_to_mesh" value="meshes/XM540-W150-R.dae" />
+        <!-- 各辺の中点が原点となるように変換 -->
 		<xacro:property name="visual_origin"> <origin xyz="${0} ${0.0386} ${0}" rpy="${-pi/2} 0 ${pi}" /> </xacro:property>
+        <!-- 各辺の中点を原点としたときのホーン中心の座標 -->
 		<xacro:property name="L_x_hone" value="${ 0.0/1000}" /> <!-- unit [m] --> <!-- converted from [mm] -->
 		<xacro:property name="L_y_hone" value="${15.5/1000}" /> <!-- unit [m] --> <!-- converted from [mm] -->
@@ -20,15 +29,18 @@
 			                                                                       izz="${ 60707.131/1000000000}" />
 		</xacro:property>
-		<joint name="XM540_base_joint_" type="fixed">
+		<joint name="${joint_name}_XM540_base_connector_" type="fixed">
 			<parent link="${parent}"/>
-			<child link="dynx_XM540"/>
+			<child link="${joint_name}_dynx_XM540"/>
 			<xacro:if value="${fixed_plane == 'bottom'}">
-				<origin xyz="${0} ${0} ${W_y/2}" rpy="${pi/2} ${0} ${0}"/> <!-- 回転が先 -->
+				<origin xyz="${0} ${0} ${W_y/2}" rpy="${pi/2} ${0} ${fixed_angle}"/> <!-- 回転が先 -->
 			</xacro:if>
 			<xacro:if value="${fixed_plane == 'top'}">
-				<origin xyz="${0} ${0} ${-W_y/2}" rpy="${pi/2} ${0} ${0}"/> <!-- 回転が先 -->
+				<origin xyz="${0} ${0} ${-W_y/2}" rpy="${pi/2} ${0} ${fixed_angle}"/> <!-- 回転が先 -->
+			</xacro:if>
+			<xacro:if value="${fixed_plane == 'back'}">
+				<origin xyz="${0} ${0} ${W_z/2}" rpy="${0} ${0} ${fixed_angle}"/> <!-- 回転が先 -->
 			</xacro:if>
 		</joint>
-		<link name="dynx_XM540">
+		<link name="${joint_name}_dynx_XM540">
 			<inertial>
 				<origin xyz="0 0 0" rpy="0 0 0"/>
@@ -53,7 +65,7 @@
 			</collision>
 		</link>
-		<joint name="${child}_joint" type="fixed">
-			<parent link="dynx_XM540"/>
-			<child link="dynx_XM540_hone"/>
+		<joint name="${joint_name}_joint" type="continuous">
+			<parent link="${joint_name}_dynx_XM540"/>
+			<child link="${joint_name}_dynx_XM540_hone"/>
 			<origin xyz="${L_x_hone} ${L_y_hone} ${L_z_hone}" rpy="0 0 0"/>
 			<axis xyz="0 0 1"/>
@@ -61,7 +73,16 @@
 			<limit velocity="${no_load_speed}" effort="${stall_torque}" />
 		</joint>
-		<link name="dynx_XM540_hone" />
-		<joint name="XM540_hone_joint_" type="fixed">
-			<parent link="dynx_XM540_hone"/>
+		<link name="${joint_name}_dynx_XM540_hone" >
+			<inertial>
+			<origin xyz="0 0 0" rpy="0 0 0" />
+			<mass value="0.00001" />
+			<inertia
+				ixx="0.00001" ixy="0.0" ixz="0.0"
+				iyy="0.00001" iyz="0.0"
+				izz="0.00001" />
+			</inertial>
+		</link>
+		<joint name="${joint_name}_XM540_hone_joint_" type="fixed">
+			<parent link="${joint_name}_dynx_XM540_hone"/>
 			<child link="${child}"/>
 			<xacro:if value="${center_child}">
@@ -73,3 +94,38 @@
 		</joint>
 	</xacro:macro>
+    <!-- フレームFR12_S102Kを装着したver -->
+    <xacro:macro name="servo_XM540_FR12_S102K" params="name:='__defalut__' parent child fixed_plane:=bottom fixed_angle:=0 center_child:=false">
+        <xacro:property name="path_to_mesh" value="meshes/fr12_s102.stl" />
+        <!-- 各辺の中点が原点となるように変換 -->
+		<xacro:property name="visual_origin"> <origin xyz="${0} ${0} ${19.5/1000-offset}" rpy="${pi} ${0} ${pi/2}" /> </xacro:property>
+		<xacro:property name="offset"  value="${5.25/1000}" /> <!-- unit [kg] --> <!-- converted from [g] -->
+		<xacro:property name="mass"  value="${165/1000}" /> <!-- unit [kg] --> <!-- converted from [g] -->
+		<xacro:property name="inertia"> <!-- unit [kg*m^@] --> <!-- converted from [g*mm^2] -->
+			<inertia ixx="${ 1999.314/1000000000}"  ixy="${    0.0  /1000000000}" ixz="${     0.0  /1000000000}"
+			                                        iyy="${ 2690.794/1000000000}" iyz="${     0.0  /1000000000}"
+			                                                                       izz="${ 1440.750/1000000000}" />
+		</xacro:property>
+        <joint name="${name}_XM540_FR12_S102K_connect_" type="fixed">
+			<parent link="${parent}"/>
+			<child link="${name}_fr_FR12_S102K_"/>
+            <origin xyz="${0} ${0} ${offset}" rpy="${0} ${0} ${fixed_angle}"/> <!-- 回転が先 -->
+		</joint>
+		<link name="${name}_fr_FR12_S102K_">
+			<inertial>
+				<origin xyz="0 0 0" rpy="0 0 0"/>
+				<mass value="${mass}"/>
+				<xacro:insert_block name="inertia"/>
+			</inertial>
+			<visual>
+				<xacro:insert_block name="visual_origin"/>
+				<geometry>
+					<mesh filename="package://dynamixel_description/${path_to_mesh}" />
+				</geometry>
+				<material name="gray">
+					<color rgba="0.8 0.8 0.8 0.5"/>
+				</material>
+			</visual>
+		</link>
+    	<xacro:servo_XM540 name="${name}" parent="${name}_fr_FR12_S102K_" child="${child}" center_child="${center_child}" fixed_plane="${fixed_plane}"/>
+	</xacro:macro>
 </robot>

File: ros/dynamixel_description/urdf/test_XM540_servo.urdf.xacro (robot description, xacro)
@@ -7,10 +7,10 @@
 			<origin xyz="0 0 0" rpy="0 0 0"/>
 			<geometry>
-				<cylinder length="0.001" radius="0.01"/>
+				<box size="0.05 0.08 0.001"/>
 			</geometry>
 			<material name="orange"/>
 		</visual>
 	</link>
-	<xacro:servo_XM540 parent="base" child="hone" center_child="false" />
+	<xacro:servo_XM540 parent="base" child="hone" center_child="true" fixed_plane="back"/>
 	<link name="hone">
 		<visual>
@@ -28,3 +28,8 @@
 		<material>Gazebo/Red</material>
 	</gazebo>
+    <!--ros_controlプラグインをロード-->
+    <gazebo>
+        <plugin name="control" filename="libgazebo_ros_control.so">
+        </plugin>
+    </gazebo>
 </robot>
