Commit message: fix typo

File: ros/dynamixel_description/urdf/_2XC430.gazebo.xacro (robot description, xacro)
@@ -1,7 +1,18 @@
 <?xml version="1.0"?>
 <!-- あとでdynamixel descriptionを作ってそこにれる -->
-<robot name=" dynamixel-2XC430" xmlns:xacro="http://ros.org/wiki/xacro">\
-	<!--あとでgazebo.xacroに入れる-->
-	<gazebo reference="dynx_2XC430">
+<robot name="dynamixel-2XC430" xmlns:xacro="http://ros.org/wiki/xacro">\
+	<!-- Transmission macro -->
+	<xacro:macro name="SimpleTransmissionPosition" params="joint motor">
+		<transmission name="tran_${joint}">
+			<type>transmission_interface/SimpleTransmission</type>
+			<joint name="${joint}">
+			    <hardwareInterface>hardware_interface/PositionJointInterface</hardwareInterface>
+			</joint>
+			<actuator name="${motor}">
+			    <mechanicalReduction>1</mechanicalReduction>
+			</actuator>
+		</transmission>
+	</xacro:macro>
+	<gazebo reference="${parent_joint_name}_${child_joint_name}_dynx_2XC430">
 		<mu1>0.1</mu1>
 		<mu2>0.1</mu2>
@@ -13,3 +24,11 @@
 		<material>Gazebo/Gray</material>
 	</gazebo>
+	<xacro:SimpleTransmissionPosition motor="${parent_joint_name}_dynx_motor1" joint="${parent_joint_name}_joint" />
+	<xacro:SimpleTransmissionPosition motor="${child_joint_name}_dynx_motor2" joint="${child_joint_name}_joint" />
+    <!--ros_controlプラグインをロード-->
+    <gazebo>
+      <plugin name="joint_state_publisher" filename="libgazebo_ros_joint_state_publisher.so">
+         <jointName>${parent_joint_name}_joint, ${child_joint_name}_joint</jointName>
+      </plugin>
+    </gazebo>
 </robot>

File: ros/dynamixel_description/urdf/_2XC430.urdf.xacro (robot description, xacro)
@@ -2,6 +2,18 @@
 <!-- あとでdynamixel descriptionを作ってそこにれる -->
 <robot name=" dynamixel-2XC430" xmlns:xacro="http://ros.org/wiki/xacro">\
-	<xacro:macro name="servo_2XC430" params="parent child center_parent:=false center_child:=false">
-	   <xacro:include filename="$(find dynamixel_description)/urdf/_2XC430.gazebo.xacro"/>
+	<xacro:macro name="servo_2XC430" params="name_parent:='__default__' parent name_child:='__default__' child center_parent:=false center_child:=false">
+        <xacro:if value="${name_parent == '__default__'}">
+		    <xacro:property name="parent_joint_name" value="${parent}" />
+        </xacro:if>
+        <xacro:unless value="${name_parent == '__default__'}">
+		    <xacro:property name="parent_joint_name" value="${name_parent}" />
+        </xacro:unless>
+        <xacro:if value="${name_child == '__default__'}">
+		    <xacro:property name="child_joint_name" value="${child}" />
+        </xacro:if>
+        <xacro:unless value="${name_child == '__default__'}">
+		    <xacro:property name="child_joint_name" value="${name_child}" />
+        </xacro:unless>
+        <xacro:include filename="$(find dynamixel_description)/urdf/_2XC430.gazebo.xacro"/>
 		<xacro:property name="path_to_mesh" value="meshes/2XC430-W250-T.stl" />
 		<xacro:property name="visual_origin"> <origin xyz="${0} ${0} ${0}" rpy="${0} ${0} ${0}" /> </xacro:property>
@@ -9,5 +21,5 @@
 		<xacro:property name="L_y_yaw" value="${12/1000}" /> <!-- unit [m] --> <!-- converted from [mm] -->
 		<xacro:property name="L_z_yaw" value="${19/1000}" /> <!-- unit [m] --> <!-- converted from [mm] -->
-		<xacro:property name="L_x_pitch" value="${ L_z_yaw}" /> <!-- unit [m] -->
+		<xacro:property name="L_x_pitch" value="${-L_z_yaw}" /> <!-- unit [m] -->
 		<xacro:property name="L_y_pitch" value="${-L_y_yaw}" /> <!-- unit [m] -->
 		<xacro:property name="L_z_pitch" value="${ L_x_yaw}" /> <!-- unit [m] -->
@@ -23,7 +35,7 @@
 			                                izz="0.11" />
 		</xacro:property> <!--todo, this is not correct-->
-		<joint name="2XC430_yaw_joint_" type="fixed">
+		<joint name="${parent_joint_name}_2XC430_yaw_fixed_" type="fixed">
 			<parent link="${parent}"/>
-			<child link="dynx_2XC430_hone_yaw"/>
+			<child link="${parent_joint_name}_dynx_2XC430_hone_yaw"/>
 			<xacro:if value="${center_parent}">
 				<origin xyz="0 0 ${-L_z_yaw}" rpy="0 0 0"/>
@@ -33,22 +45,29 @@
 			</xacro:unless>
 		</joint>
-		<link name="dynx_2XC430_hone_yaw" />
-		<joint name="${parent}_joint" type="fixed">
-			<parent link="dynx_2XC430_hone_yaw"/>
-			<child link="dynx_2XC430"/>
-			<origin xyz="${L_x_yaw} ${L_y_yaw} ${L_z_yaw}" rpy="${pi} 0 0"/>
-			<!--6.3879[rad/sec]=61[rev/min], 1.5[Nm]-->
+		<link name="${parent_joint_name}_dynx_2XC430_hone_yaw">
+			<inertial>
+				<origin xyz="0 0 0" rpy="0 0 0" />
+				<mass value="0.00001" />
+				<inertia
+					ixx="0.00001" ixy="0.0" ixz="0.0"
+					iyy="0.00001" iyz="0.0"
+					izz="0.00001" />
+			</inertial>
+		</link>
+		<joint name="${parent_joint_name}_joint" type="continuous">
+			<parent link="${parent_joint_name}_dynx_2XC430_hone_yaw"/>
+			<child link="${parent_joint_name}_${child_joint_name}_dynx_2XC430"/>
 			<axis xyz="0 0 1"/>
 			<dynamics damping="0.1"/>
 			<limit velocity="${no_load_speed}" effort="${stall_torque}" />
 		</joint>
-		<link name="dynx_2XC430">
+		<link name="${parent_joint_name}_${child_joint_name}_dynx_2XC430">
 			<inertial>
-				<origin xyz="0 0 0" rpy="0 0 0"/>
+			    <origin xyz="${L_x_yaw} ${L_y_yaw} ${L_z_yaw}" rpy="${pi} 0 0"/>
 				<mass value="${mass}"/>
 				<xacro:insert_block name="inertia"/>
 			</inertial>
 			<visual>
-				<xacro:insert_block name="visual_origin"/>
+                <origin xyz="${L_x_yaw} ${L_y_yaw} ${L_z_yaw}" rpy="${pi} 0 0"/>
 				<geometry>
 					<mesh filename="package://dynamixel_description/${path_to_mesh}" />
@@ -59,5 +78,5 @@
 			</visual>
 			<collision>
-				<origin xyz="0 0 0" rpy="0 0 0"/>
+			   <origin xyz="${L_x_yaw} ${L_y_yaw} ${L_z_yaw}" rpy="${pi} 0 0"/>
 				<geometry>
 					<box size="${W_x} ${W_y} ${W_z}"/>
@@ -66,22 +85,30 @@
 			</collision>
 		</link>
-		<joint name="${child}_joint" type="fixed">
-			<parent link="dynx_2XC430"/>
-			<child link="dynx_2XC430_hone_pitch"/>
-			<origin xyz="${L_x_pitch} ${L_y_pitch} ${L_z_pitch}" rpy="0 ${pi/2} 0"/>
-			<!--6.3879[rad/sec]=61-->
-			<axis xyz="0 0 1"/>
+		<joint name="${child_joint_name}_joint" type="continuous">
+			<parent link="${parent_joint_name}_${child_joint_name}_dynx_2XC430"/>
+			<child link="${child_joint_name}_dynx_2XC430_hone_pitch"/>
+			<origin xyz="${L_x_yaw-L_x_pitch} ${L_y_yaw-L_y_pitch} ${L_z_yaw-L_z_pitch}" rpy="${pi} 0 0"/>
+			<axis xyz="1 0 0"/>
 			<dynamics damping="0.1"/>
 			<limit velocity="${no_load_speed}" effort="${stall_torque}" />
 		</joint>
-		<link name="dynx_2XC430_hone_pitch" />
-		<joint name="2XC430_pitch_joint_" type="fixed">
-			<parent link="dynx_2XC430_hone_pitch"/>
+		<link name="${child_joint_name}_dynx_2XC430_hone_pitch">
+			<inertial>
+			<origin xyz="0 0 0" rpy="0 0 0" />
+			<mass value="0.00001" />
+			<inertia
+				ixx="0.00001" ixy="0.0" ixz="0.0"
+				iyy="0.00001" iyz="0.0"
+				izz="0.00001" />
+			</inertial>
+		</link>
+		<joint name="${child_joint_name}_2XC430_pitch_fixed_" type="fixed">
+			<parent link="${child_joint_name}_dynx_2XC430_hone_pitch"/>
 			<child link="${child}"/>
 			<xacro:if value="${center_child}">
-				<origin xyz="0 0 ${-L_x_pitch}" rpy="0 0 0"/>
+				<origin xyz="${L_x_pitch} 0 0" rpy="0 ${pi/2} 0"/>
 			</xacro:if>
 			<xacro:unless value="${center_child}">
-				<origin xyz="0 0 0" rpy="0 0 0"/>
+				<origin xyz="0 0 0" rpy="0 ${pi/2} 0"/>
 			</xacro:unless>
 		</joint>

File: ros/dynamixel_description/urdf/_2XL430.gazebo.xacro (robot description, xacro)
@@ -14,5 +14,5 @@
 		</transmission>
 	</xacro:macro>
-	<gazebo reference="dynx_2XL430">
+	<gazebo reference="${parent_joint_name}_${child_joint_name}_dynx_2XL430">
 		<mu1>0.1</mu1>
 		<mu2>0.1</mu2>
@@ -24,10 +24,10 @@
 		<material>Gazebo/Gray</material>
 	</gazebo>
-	<xacro:SimpleTransmissionPosition motor="dynx_motor1" joint="${parent}_joint" />
-	<xacro:SimpleTransmissionPosition motor="dynx_motor2" joint="${child}_joint" />
+	<xacro:SimpleTransmissionPosition motor="${parent_joint_name}_dynx_motor1" joint="${parent_joint_name}_joint" />
+	<xacro:SimpleTransmissionPosition motor="${child_joint_name}_dynx_motor2" joint="${child_joint_name}_joint" />
     <!--ros_controlプラグインをロード-->
     <gazebo>
       <plugin name="joint_state_publisher" filename="libgazebo_ros_joint_state_publisher.so">
-         <jointName>${parent}_joint, ${child}_joint</jointName>
+         <jointName>${parent_joint_name}_joint, ${child_joint_name}_joint</jointName>
       </plugin>
     </gazebo>

File: ros/dynamixel_description/urdf/_2XL430.urdf.xacro (robot description, xacro)
@@ -2,6 +2,18 @@
 <!-- あとでdynamixel descriptionを作ってそこにれる -->
 <robot name=" dynamixel-2XL430" xmlns:xacro="http://ros.org/wiki/xacro">\
-	<xacro:macro name="servo_2XL430" params="parent child center_parent:=false center_child:=false">
-	   <xacro:include filename="$(find dynamixel_description)/urdf/_2XL430.gazebo.xacro"/>
+	<xacro:macro name="servo_2XL430" params="name_parent:='__default__' parent name_child:='__default__' child center_parent:=false center_child:=false">
+        <xacro:if value="${name_parent == '__default__'}">
+		    <xacro:property name="parent_joint_name" value="${parent}" />
+        </xacro:if>
+        <xacro:unless value="${name_parent == '__default__'}">
+		    <xacro:property name="parent_joint_name" value="${name_parent}" />
+        </xacro:unless>
+        <xacro:if value="${name_child == '__default__'}">
+		    <xacro:property name="child_joint_name" value="${child}" />
+        </xacro:if>
+        <xacro:unless value="${name_child == '__default__'}">
+		    <xacro:property name="child_joint_name" value="${name_child}" />
+        </xacro:unless>
+        <xacro:include filename="$(find dynamixel_description)/urdf/_2XL430.gazebo.xacro"/>
 		<xacro:property name="path_to_mesh" value="meshes/2XL430-W250-T.stl" />
 		<xacro:property name="visual_origin"> <origin xyz="${0} ${0} ${0}" rpy="${0} ${0} ${0}" /> </xacro:property>
@@ -23,7 +35,7 @@
 			                                izz="0.11" />
 		</xacro:property> <!--todo, this is not correct-->
-		<joint name="2XL430_yaw_joint_" type="fixed">
+		<joint name="${parent_joint_name}_2XL430_yaw_fixed_" type="fixed">
 			<parent link="${parent}"/>
-			<child link="dynx_2XL430_hone_yaw"/>
+			<child link="${parent_joint_name}_dynx_2XL430_hone_yaw"/>
 			<xacro:if value="${center_parent}">
 				<origin xyz="0 0 ${-L_z_yaw}" rpy="0 0 0"/>
@@ -33,22 +45,22 @@
 			</xacro:unless>
 		</joint>
-		<link name="dynx_2XL430_hone_yaw">
+		<link name="${parent_joint_name}_dynx_2XL430_hone_yaw">
 			<inertial>
-			<origin xyz="0 0 0" rpy="0 0 0" />
-			<mass value="0.00001" />
-			<inertia
-				ixx="0.00001" ixy="0.0" ixz="0.0"
-				iyy="0.00001" iyz="0.0"
-				izz="0.00001" />
+				<origin xyz="0 0 0" rpy="0 0 0" />
+				<mass value="0.00001" />
+				<inertia
+					ixx="0.00001" ixy="0.0" ixz="0.0"
+					iyy="0.00001" iyz="0.0"
+					izz="0.00001" />
 			</inertial>
 		</link>
-		<joint name="${parent}_joint" type="continuous">
-			<parent link="dynx_2XL430_hone_yaw"/>
-			<child link="dynx_2XL430"/>
+		<joint name="${parent_joint_name}_joint" type="continuous">
+			<parent link="${parent_joint_name}_dynx_2XL430_hone_yaw"/>
+			<child link="${parent_joint_name}_${child_joint_name}_dynx_2XL430"/>
 			<axis xyz="0 0 1"/>
 			<dynamics damping="0.1"/>
 			<limit velocity="${no_load_speed}" effort="${stall_torque}" />
 		</joint>
-		<link name="dynx_2XL430">
+		<link name="${parent_joint_name}_${child_joint_name}_dynx_2XL430">
 			<inertial>
 			    <origin xyz="${L_x_yaw} ${L_y_yaw} ${L_z_yaw}" rpy="${pi} 0 0"/>
@@ -66,5 +78,5 @@
 			</visual>
 			<collision>
-			    <origin xyz="${L_x_yaw} ${L_y_yaw} ${L_z_yaw}" rpy="${pi} 0 0"/>
+			   <origin xyz="${L_x_yaw} ${L_y_yaw} ${L_z_yaw}" rpy="${pi} 0 0"/>
 				<geometry>
 					<box size="${W_x} ${W_y} ${W_z}"/>
@@ -73,7 +85,7 @@
 			</collision>
 		</link>
-		<joint name="${child}_joint" type="continuous">
-			<parent link="dynx_2XL430"/>
-			<child link="dynx_2XL430_hone_pitch"/>
+		<joint name="${child_joint_name}_joint" type="continuous">
+			<parent link="${parent_joint_name}_${child_joint_name}_dynx_2XL430"/>
+			<child link="${child_joint_name}_dynx_2XL430_hone_pitch"/>
 			<origin xyz="${L_x_yaw-L_x_pitch} ${L_y_yaw-L_y_pitch} ${L_z_yaw-L_z_pitch}" rpy="${pi} 0 0"/>
 			<axis xyz="1 0 0"/>
@@ -81,5 +93,5 @@
 			<limit velocity="${no_load_speed}" effort="${stall_torque}" />
 		</joint>
-		<link name="dynx_2XL430_hone_pitch">
+		<link name="${child_joint_name}_dynx_2XL430_hone_pitch">
 			<inertial>
 			<origin xyz="0 0 0" rpy="0 0 0" />
@@ -91,6 +103,6 @@
 			</inertial>
 		</link>
-		<joint name="2XL430_pitch_joint_" type="fixed">
-			<parent link="dynx_2XL430_hone_pitch"/>
+		<joint name="${child_joint_name}_2XL430_pitch_fixed_" type="fixed">
+			<parent link="${child_joint_name}_dynx_2XL430_hone_pitch"/>
 			<child link="${child}"/>
 			<xacro:if value="${center_child}">

File: ros/dynamixel_description/urdf/test_2XC430_servo.urdf.xacro (robot description, xacro)
@@ -22,5 +22,5 @@
 		</visual>
 	</link>
-	<gazebo reference="base">
+\	<gazebo reference="base">
 		<material>Gazebo/Orange</material>
 	</gazebo>
@@ -28,3 +28,8 @@
 		<material>Gazebo/Red</material>
 	</gazebo>
+    <!--ros_controlプラグインをロード-->
+    <gazebo>
+        <plugin name="control" filename="libgazebo_ros_control.so">
+        </plugin>
+    </gazebo>
 </robot>

File: ros/dynamixel_description/urdf/test_2XL430_servo.urdf.xacro (robot description, xacro)
@@ -12,5 +12,5 @@
 		</visual>
 	</link>
-	<xacro:servo_2XL430 parent="base" center_parent="true" child="hone" center_child="true" />
+	<xacro:servo_2XL430 parent="base" center_parent="false" child="hone" center_child="true" />
 	<link name="hone">
 		<visual>
